Commit message: Lower base_link Z-height from wheel axie height to ground level

File: urdf/phoebe.urdf.xacro (robot description, xacro)
@@ -25,5 +25,5 @@
   <link name="base_link">
     <visual>
-      <origin xyz="${body_rect_length/2 - body_center_to_cylinder} 0 ${body_height/2 - body_center_to_bottom}" rpy="0 0 0"/>
+      <origin xyz="${body_rect_length/2 - body_center_to_cylinder} 0 ${body_height/2 - body_center_to_bottom + wheel_diameter/2}" rpy="0 0 0"/>
       <geometry>
         <box size="${body_rect_length} ${body_width} ${body_height}"/>
@@ -32,5 +32,5 @@
     </visual>
     <visual>
-      <origin xyz="${-body_center_to_cylinder} 0 ${body_height/2 - body_center_to_bottom}" rpy="0 0 0"/>
+      <origin xyz="${-body_center_to_cylinder} 0 ${body_height/2 - body_center_to_bottom + wheel_diameter/2}" rpy="0 0 0"/>
       <geometry>
         <cylinder radius="${body_width/2}" length="${body_height}"/>
@@ -66,5 +66,5 @@
       <parent link="base_link" />
       <child link="wheel_${side}" />
-      <origin xyz="0 ${reflect * wheel_base/2} 0" rpy="0 0 0" />
+      <origin xyz="0 ${reflect * wheel_base/2} ${wheel_diameter/2}" rpy="0 0 0" />
     </joint>
   </xacro:macro>

Commit message: Add color tint to stand out against gray map

File: urdf/phoebe.urdf.xacro (robot description, xacro)
@@ -14,12 +14,12 @@
   <xacro:property name="wheel_base" value="0.215" />
   <xacro:property name="wheel_diameter" value="0.067" />
-  <material name="blue">
-    <color rgba="0 0 0.8 1"/>
+  <material name="neato">
+    <color rgba="0.3 0.2 0.2 1"/>
   </material>
-  <material name="black">
-    <color rgba="0 0 0 1"/>
+  <material name="wheel">
+    <color rgba="0.3 0.2 0.2 1"/>
   </material>
-  <material name="white">
-    <color rgba="1 1 1 1"/>
+  <material name="body">
+    <color rgba="0.6 0.6 0.7 1"/>
   </material>
   <link name="base_link">
@@ -29,5 +29,5 @@
         <box size="${body_rect_length} ${body_width} ${body_height}"/>
       </geometry>
-      <material name="white" />
+      <material name="body" />
     </visual>
     <visual>
@@ -36,5 +36,5 @@
         <cylinder radius="${body_width/2}" length="${body_height}"/>
       </geometry>
-      <material name="white" />
+      <material name="body" />
     </visual>
   </link>
@@ -44,5 +44,5 @@
         <cylinder radius="${neato_diameter/2}" length="${neato_height}"/>
       </geometry>
-      <materual name="blue" />
+      <material name="neato" />
     </visual>
   </link>
@@ -59,5 +59,5 @@
           <cylinder radius="${wheel_diameter/2}" length="${wheel_width}"/>
         </geometry>
-        <material name="black" />
+        <material name="wheel" />
       </visual>
     </link>

Commit message: Fix problems exposed trying to use URDF in RViz * Neato laser needs to be moved up to compensate for   base_link moving down to ground level. * Neato laser needs to rotate 180 degrees to match   sensor mount location * A sphere was added to correspond to caster wheel. * Drive wheels are "fixed" for now, at least until we can   publish wheel angles.

File: urdf/phoebe.urdf.xacro (robot description, xacro)
@@ -50,5 +50,5 @@
     <parent link="base_link"/>
     <child link="neato_laser"/>
-    <origin xyz="${neato_offset_x} ${neato_offset_y} ${neato_offset_z}"/>
+    <origin xyz="${neato_offset_x} ${neato_offset_y} ${neato_offset_z + wheel_diameter/2}" rpy="0 0 ${pi}" />
   </joint>
   <xacro:macro name="wheel" params="side reflect">
@@ -62,5 +62,5 @@
       </visual>
     </link>
-    <joint name="base_wheel_${side}_joint" type="continuous">
+    <joint name="base_wheel_${side}_joint" type="fixed"> <!-- TODO: type="continuous" when we read encoder data and publish wheel angle -->
       <axis xyz="0 1 0" rpy="0 0 0" />
       <parent link="base_link" />
@@ -71,3 +71,16 @@
   <xacro:wheel side="left" reflect="1" />
   <xacro:wheel side="right" reflect="-1" />
+  <link name="wheel_caster">
+    <visual>
+      <geometry>
+        <sphere radius="${wheel_diameter/2}" />
+      </geometry>
+      <material name="wheel" />
+    </visual>
+  </link>
+  <joint name="base_caster" type="fixed">
+    <parent link="base_link" />
+    <child link="wheel_caster" />
+    <origin xyz="${-body_center_to_cylinder-body_width/2+wheel_diameter/2} 0 ${wheel_diameter/2}" />
+  </joint>
 </robot>
